Commit message: use unlimited for calibration and has megvii demo

File: chessbot_description/urdf/chessbot.urdf.xacro (robot description, xacro)
@@ -2,5 +2,5 @@
 <robot xmlns:xacro="http://www.ros.org/wiki/xacro" name="chessbot" >
   <property name="M_PI" value="3.14159265359" />
-  <property name="kinect_prefix1" value=""/>
+  <!--<property name="kinect_prefix1" value=""/>-->
   <property name="robot_prefix1" value=""/>
   <!-- common stuff -->
@@ -14,10 +14,16 @@
   <!-- rg2 gripper -->
   <xacro:include filename="$(find chessbot_description)/urdf/rg2.urdf.xacro" />
+  <!-- aruco board -->
+  <xacro:include filename="$(find chessbot_description)/urdf/aruco.urdf.xacro"/>
   <!-- arm -->
   <xacro:ur5_robot prefix="${robot_prefix1}" joint_limited="false"/>
+  <!-- 3D sensor -->
+  <!--<xacro:sensor_kinect prefix="${robot_prefix1}"/>-->
   <!-- arm extras -->
-  <xacro:support_base prefix="${robot_prefix1}" kinect_prefix="${kinect_prefix1}"/>
+  <xacro:support_base prefix="${robot_prefix1}"/>
   <!-- rg2 pipe -->
   <xacro:rg2 prefix="${robot_prefix1}"/>
+  <!-- aruco board -->
+  <xacro:aruco prefix="${robot_prefix1}"/>
   <!-- world will be root link-->
   <link name="world" />

File: chessbot_description/urdf/chessbot_limited.urdf.xacro (robot description, xacro)
@@ -2,5 +2,5 @@
 <robot xmlns:xacro="http://www.ros.org/wiki/xacro" name="chessbot" >
   <property name="M_PI" value="3.14159265359" />
-  <property name="kinect_prefix1" value=""/>
+  <!--<property name="kinect_prefix1" value=""/>-->
   <property name="robot_prefix1" value=""/>
   <!-- common stuff -->
@@ -14,4 +14,6 @@
   <!-- rg2 gripper -->
   <xacro:include filename="$(find chessbot_description)/urdf/rg2.urdf.xacro" />
+  <!-- aruco board -->
+  <xacro:include filename="$(find chessbot_description)/urdf/aruco.urdf.xacro"/>
   <!-- arm -->
   <!-- we limit the first 3 joints to get a limited action space -->
@@ -24,8 +26,12 @@
     wrist_3_lower_limit="${-pi}" wrist_3_upper_limit="${pi}"
   />
+    <!-- 3D sensor -->
+  <!--<xacro:sensor_kinect prefix="${robot_prefix1}"/>-->
   <!-- arm extras -->
-  <xacro:support_base prefix="${robot_prefix1}" kinect_prefix="${kinect_prefix1}"/>
+  <xacro:support_base prefix="${robot_prefix1}"/>
   <!-- rg2 pipe -->
   <xacro:rg2 prefix="${robot_prefix1}"/>
+  <!-- aruco board -->
+  <xacro:aruco prefix="${robot_prefix1}"/>
   <!-- world will be root link-->
   <link name="world" />

File: chessbot_description/urdf/support_base.urdf.xacro (robot description, xacro)
@@ -2,5 +2,5 @@
 <!-- xacro for extras components mounted on the manipulator -->
 <robot name="support_base" xmlns:xacro="http://ros.org/wiki/xacro">
-  <xacro:macro name="support_base" params="prefix kinect_prefix">
+  <xacro:macro name="support_base" params="prefix">
     <link name="${prefix}base_chassis">
       <visual>
